File: hardware/dc-v2.kicad_pcb (KiCad board)
At the start: 2 copper layers, 40 x 40 mm, 37 parts, among them P1 black, P101 CON-SENSOR2, P102 DEBUG, P103 BOOT, P2 green, Q1 FDS8449, U1 MC33926, U101 XMC1XXX, U103 DRILL, U104 DRILL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

Commit message: ready for prototype
Parts:
- added D3: red, kicad-libraries:D0603F, F.Cu at (131.3, 101.8)
- added Fiducial_Mark: VAL**, kicad-libraries:Fiducial_Mark, F.Cu at (132.0, 138.0)
- added Fiducial_Mark: VAL**, kicad-libraries:Fiducial_Mark, F.Cu at (107.0, 138.0)
- added Fiducial_Mark: VAL**, kicad-libraries:Fiducial_Mark, F.Cu at (130.0, 107.0)
- added G***: LOGO, kicad-libraries:Logo_31x31, F.Cu at (133.9, 106.9)
- added R7: 1k, kicad-libraries:R0603F, F.Cu at (130.0, 101.8)
- moved VAL 0.10 mm to (112.8, 120.0)
Routing:
- net Net-(R7-Pad1): track 0.00 -> 22.6 mm, vias 0 -> 2
- net 3V3: track 48.0 -> 54.4 mm
- net Net-(D3-Pad2): track 0.00 -> 1.35 mm
- net VCC: track 21.1 -> 20.8 mm, vias 11 -> 63
- net GND: track 22.8 -> 22.9 mm, vias 23 -> 21
- net AGND: vias 9 -> 114
Other:
- board text added: "+"
- board text added: "-"
- board text added: "DC 2.0"
- board text added: "Error"
- board text added: "Input 6-28V"
- board text added: "Output"
- board text added: "Status"
- board text added: "tinkerforge.com"
